File: hardware_design/labRF_Kicad/328p_design/328p_design.kicad_sch (KiCad schematic)
At the start: 45 parts, among them J1 select_rotary, J10 pwmC, J11 pwrIn, J2 mode_rotary, J3 lcd_socket, J4 comms, J5 si5351, J6 clk0, J7 clk2, J8 bias_pot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

Commit message: Upgraded Schematic to 9V reference
Parts:
- removed C9: 10n, Capacitor_THT:C_Disc_D5.0mm_W2.5mm_P2.50mm, symbol Device:C
- removed Q2: BC547, Package_TO_SOT_THT:TO-92_Inline, symbol Transistor_BJT:BC547
- removed R3: 10k, Resistor_THT:R_Axial_DIN0207_L6.3mm_D2.5mm_P10.16mm_Horizontal, symbol Device:R
- added C15: 10n, Capacitor_THT:C_Disc_D5.0mm_W2.5mm_P2.50mm, symbol Device:C
- added Q2, Q5: BC557, Package_TO_SOT_THT:TO-92_Inline, symbol Transistor_BJT:BC557
- added Q6: BC547, Package_TO_SOT_THT:TO-92_Inline, symbol Transistor_BJT:BC547
- added R10, R6, R8: 10k, Resistor_THT:R_Axial_DIN0207_L6.3mm_D2.5mm_P10.16mm_Horizontal, symbol Device:R
- added R7, R9: 1k, Resistor_THT:R_Axial_DIN0207_L6.3mm_D2.5mm_P10.16mm_Horizontal, symbol Device:R
Connections:
- net +5V: no longer Q4.1 (C), R5.2
- net GND: now also Q1.3 (E), C15.2, Q6.3 (E)
- net bias: now also R8.1
- net at C13.2, C14.1, C7.2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: now also Q2.3 (E), Q5.3 (E); no longer Q1.1 (C)
- net +9V: now reaches C10.2, J11.1 (Pin_1), U4.1 (IN)
- net +9V: now also Q4.1 (C), R5.2, R7.2, R9.2
- net at L2.1: now also Q2.1 (C)
- net at L1.1: now also Q5.1 (C); no longer Q1.3 (E)
- new net: Q5.2 (B), R6.2
- new net: Q1.1 (C), R6.1, R7.1
- new net: Q6.1 (C), R10.1, R9.1
- new net: Q2.2 (B), R10.2
- new net: C15.1, Q6.2 (B), R8.2
Other:
- moved on the sheet: BZ1, C6, J5, Q1, Q3, R2, R4
