File: hardware_design/labRF_Kicad/labRF/labRF.kicad_sch (KiCad schematic)
At the start: 45 parts, among them J1 select_rotary, J10 pwmC, J11 pwrIn, J12 clk2, J2 mode_rotary, J3 lcd_socket, J4 comms, J5 si5351, J6 clk0, J7 clk2, J8 bias_pot, J9 pwmD, Q1 BC547, Q2 BC547, Q3 BC547, Q4 BC547, U1 CMT2119, U2 TL431LP, U3 74HC04, U4 L7805, U5 YAAJ_BluePill, Y1 26Mhz

Commit message: Finished bluepill schematics
Parts:
- removed C13: 100n, Capacitor_THT:C_Disc_D5.0mm_W2.5mm_P2.50mm, symbol Device:C
- removed C14: 100u, Capacitor_THT:CP_Radial_D8.0mm_P5.00mm, symbol Device:C_Polarized
- removed C8, C9: 10n, Capacitor_THT:C_Disc_D5.0mm_W2.5mm_P2.50mm, symbol Device:C
- removed J6: clk0, Connector_PinHeader_2.54mm:PinHeader_1x02_P2.54mm_Vertical, symbol Connector:Conn_01x02_Socket
- removed J7: clk2, Connector_PinHeader_2.54mm:PinHeader_1x02_P2.54mm_Vertical, symbol Connector:Conn_01x02_Socket
- removed J8: bias_pot, Connector:FanPinHeader_1x03_P2.54mm_Vertical, symbol Connector:Conn_01x03_Socket
- removed JP2: Jumper_2_Open, Connector_PinHeader_2.54mm:PinHeader_1x02_P2.54mm_Vertical, symbol Jumper:Jumper_2_Open
- removed Q1, Q4: BC547, Package_TO_SOT_THT:TO-92_Inline, symbol Transistor_BJT:BC547
- removed U2: TL431LP, Package_TO_SOT_THT:TO-92_Inline, symbol Reference_Voltage:TL431LP
- added C15, C16, C19: 100n, Capacitor_THT:C_Disc_D5.0mm_W2.5mm_P2.50mm, symbol Device:C
- added C17, C20: 10n, Capacitor_THT:C_Disc_D5.0mm_W2.5mm_P2.50mm, symbol Device:C
- added C18: 100u, Capacitor_THT:CP_Radial_D8.0mm_P5.00mm, symbol Device:C_Polarized
- added D1, D2: 1N4148, Diode_THT:D_DO-35_SOD27_P7.62mm_Horizontal, symbol Diode:1N4148
- added J13: bias_pot, Connector:FanPinHeader_1x03_P2.54mm_Vertical, symbol Connector:Conn_01x03_Socket
- added J14: clk0, Connector_PinHeader_2.54mm:PinHeader_1x02_P2.54mm_Vertical, symbol Connector:Conn_01x02_Socket
- added J15: clk2, Connector_PinHeader_2.54mm:PinHeader_1x02_P2.54mm_Vertical, symbol Connector:Conn_01x02_Socket
- added J6: Conn_01x03_Socket, Connector_PinHeader_2.54mm:PinHeader_1x03_P2.54mm_Vertical, symbol Connector:Conn_01x03_Socket
- added JP3, JP4: Jumper_2_Open, Connector_PinHeader_2.54mm:PinHeader_1x02_P2.54mm_Vertical, symbol Jumper:Jumper_2_Open
- added L3: 100u, Inductor_THT:L_Toroid_Vertical_L14.7mm_W8.6mm_P5.58mm_Pulse_KM-1, symbol Device:L
- added Q1, Q7, Q8: BC557, Package_TO_SOT_THT:TO-92_Inline, symbol Transistor_BJT:BC557
- added Q5, Q6, Q9: BC547, Package_TO_SOT_THT:TO-92_Inline, symbol Transistor_BJT:BC547
- added R1, R11, R8, R9: 10k, Resistor_THT:R_Axial_DIN0207_L6.3mm_D2.5mm_P10.16mm_Horizontal, symbol Device:R
- added R10, R6, R7: 1k, Resistor_THT:R_Axial_DIN0207_L6.3mm_D2.5mm_P10.16mm_Horizontal, symbol Device:R
- added R12, R13: 100k, Resistor_THT:R_Axial_DIN0207_L6.3mm_D2.5mm_P10.16mm_Horizontal, symbol Device:R
- added U2: LM358, Package_DIP:DIP-8_W7.62mm, symbol Amplifier_Operational:LM358
- added U6: TL431LP, Package_TO_SOT_THT:TO-92_Inline, symbol Reference_Voltage:TL431LP
- C4, C5: value 100n -> 10n
- C7: value 10n -> 100n
- L2: value 100u -> 200n
- R3: value 10k -> 1k
- R5: value 1k -> 10k
Connections:
- net +3V3: now also L2.2
- net +5V: no longer R5.2
- net GND: now also C4.2, C5.2, Q2.3 (E), C16.1, C17.1, C18.2, C20.1, J13.3 (Pin_3), J14.2 (Pin_2), J15.2 (Pin_2), J6.2 (Pin_2), Q6.3 (E), Q9.3 (E), R12.2, R13.2, U2.4 (V-), U6.2 (A)
- net chanE: now also L2.1
- net clk0: now also C15.1; no longer C4.1
- net clk2: now also C19.1; no longer C5.1
- net at Q2.1 (C): now also R2.1, R3.1; no longer C7.2
- net at JP1.1 (A): now also C2.2, J12.1 (Pin_1); no longer C4.2
- net +9V: now reaches C10.2, J11.1 (Pin_1), U4.1 (IN)
- net +9V: now also C7.2, R3.2, Q5.1 (C), R10.2, R6.2, R7.2, U2.8 (V+)
- net bias3: now reaches R5.1
- net bias3: now also U5.35 (PB10)
- net adc2: now reaches U5.25 (PA0)
- net adc2: now also U2.1, U2.2 (-)
- net adc1: now reaches U5.26 (PA1)
- net adc1: now also U2.6 (-), U2.7
- net bias1: now reaches U5.27 (PA2)
- net bias1: now also R1.1
- net bias2: now reaches U5.28 (PA3)
- net bias2: now also R11.1
- net at Q2.2 (B): now also C4.1, R5.2; no longer R3.2
- net at R2.2: now also Q1.2 (B); no longer C6.1
- net at L1.1: now also C16.2, C17.2, C18.1, C20.2, J13.1 (Pin_1), L3.1, Q5.3 (E)
- net at L1.2: now also Q7.3 (E), Q8.3 (E); no longer JP1.2 (B)
- removed net bias: R2.1, R3.1, U5.35 (PB10)
- new net: Q9.1 (C), R10.1, R9.1
- new net: Q9.2 (B), R11.2
- new net: Q6.1 (C), R7.1, R8.1
- new net: Q6.2 (B), R1.2
- new net: Q7.2 (B), R8.2
- new net: C15.2, J14.1 (Pin_1), JP3.1 (A)
- new net: JP3.2 (B), Q7.1 (C)
- new net: C5.1, D1.1 (K), R12.1, U2.3 (+)
- new net: C19.2, J15.1 (Pin_1), JP4.1 (A)
- new net: C6.1, D2.1 (K), R13.1, U2.5 (+)
- new net: JP1.2 (B), Q1.1 (C)
- new net: L3.2, Q1.3 (E)
- new net: D1.2 (A), J6.1 (Pin_1)
- new net: D2.2 (A), J6.3 (Pin_3)
- new net: JP4.2 (B), Q8.1 (C)
- new net: Q5.2 (B), R6.1, U6.3 (K)
- new net: J13.2 (Pin_2), U6.1 (REF)
- new net: Q8.2 (B), R9.2
- no-connect marks 14 -> 21
Other:
- company: (none) -> Suryasaradhi
- title: (none) -> RFGen
- moved on the sheet: BZ1, C2, J10, J12, J5, J9, Q3, R4, U3A, U3B, U3C, U3D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
