File: hardware_design/bluepill_design/bluepill_design.kicad_sch (KiCad schematic)
At the start: 66 parts, among them J1 select_rotary, J10 pwmC, J11 pwrIn, J12 clk2, J13 bias_pot, J14 clk0, J15 clk2, J2 mode_rotary, J3 lcd_socket, J4 comms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

Commit message: Added blue pill code
Connections:
- net +3V3: now also J1.4 (Pin_4), J2.4 (Pin_4)
- net +5V: no longer J1.4 (Pin_4), J2.4 (Pin_4)
Changed lines of the file:
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@@
 	)
 	(symbol
-		(lib_id "power:GND")
-		(at 186.69 85.09 180)
+		(lib_id "power:+3V3")
+		(at 21.59 161.29 180)
 		(unit 1)
 		(exclude_from_sim no)
@@
 		(dnp no)
 		(fields_autoplaced yes)
-		(property "Reference" "#PWR021"
-			(at 186.69 78.74 0)
+		(property "Reference" "#PWR07"
+			(at 21.59 157.48 0)
 			(effects
 				(font
@@
 			)
 		)
-		(property "Value" "GND"
-			(at 186.69 80.01 0)
+		(property "Value" "+3V3"
+			(at 21.59 166.37 0)
 			(effects
 				(font
@@
 		)
 		(property "Footprint" ""
-			(at 186.69 85.09 0)
+			(at 21.59 161.29 0)
 			(effects
 				(font
@@
 		)
 		(property "Datasheet" ""
-			(at 186.69 85.09 0)
+			(at 21.59 161.29 0)
 			(effects
 				(font
@@
 			)
 		)
-		(property "Description" "Power symbol creates a global label with name \"GND\" , ground"
-			(at 186.69 85.09 0)
+		(property "Description" "Power symbol creates a global label with name \"+3V3\""
+			(at 21.59 161.29 0)
 			(effects
 				(font
@@
 		)
 		(instances
-			(project "labRF"
+			(project "bluepill_design"
 				(path "/2343659c-5e3e-4b93-ace6-06935e396af8"
-					(reference "#PWR021")
+					(reference "#PWR07")
 					(unit 1)
 				)
@@
 	)
 	(symbol
-		(lib_id "Transistor_BJT:BC547")
-		(at 172.72 133.35 0)
-		(mirror y)
+		(lib_id "power:GND")
+		(at 186.69 85.09 180)
 		(unit 1)
 		(exclude_from_sim no)
@@
 		(dnp no)
 		(fields_autoplaced yes)
-		(property "Reference" "Q9"
-			(at 167.64 132.0799 0)
+		(property "Reference" "#PWR021"
+			(at 186.69 78.74 0)
 			(effects
 				(font
 					(size 1.27 1.27)
 				)
-				(justify left)
+				(hide yes)
 			)
 		)
-		(property "Value" "BC547"
-			(at 167.64 134.6199 0)
+		(property "Value" "GND"
+			(at 186.69 80.01 0)
 			(effects
 				(font
 					(size 1.27 1.27)
 				)
-				(justify left)
 			)
 		)
-		(property "Footprint" "Package_TO_SOT_THT:TO-92_Inline"
-			(at 167.64 135.255 0)
+		(property "Footprint" ""
+			(at 186.69 85.09 0)
 			(effects
 				(font
 					(size 1.27 1.27)
-					(italic yes)
 				)
-				(justify left)
 				(hide yes)
 			)
 		)
-		(property "Datasheet" "https://www.onsemi.com/pub/Collateral/BC550-D.pdf"
-			(at 172.72 133.35 0)
+		(property "Datasheet" ""
+			(at 186.69 85.09 0)
 			(effects
 				(font
 					(size 1.27 1.27)
 				)
-				(justify left)
 				(hide yes)
 			)
 		)
-		(property "Description" "0.1A Ic, 45V Vce, Small Signal NPN Transistor, TO-92"
-			(at 172.72 133.35 0)
+		(property "Description" "Power symbol creates a global label with name \"GND\" , ground"
+			(at 186.69 85.09 0)
 			(effects
 				(font
@@
 			)
 		)
-		(pin "3"
-		)
-		(pin "2"
-		)
 		(pin "1"
 		)
@@
 			(project "labRF"
 				(path "/2343659c-5e3e-4b93-ace6-06935e396af8"
-					(reference "Q9")
+					(reference "#PWR021")
 					(unit 1)
 				)
@@
 	)
 	(symbol
-		(lib_id "power:+5V")
-		(at 21.59 138.43 180)
+		(lib_id "Transistor_BJT:BC547")
+		(at 172.72 133.35 0)
+		(mirror y)
 		(unit 1)
 		(exclude_from_sim no)
@@
 		(dnp no)
 		(fields_autoplaced yes)
-		(property "Reference" "#PWR07"
-			(at 21.59 134.62 0)
+		(property "Reference" "Q9"
+			(at 167.64 132.0799 0)
 			(effects
 				(font
 					(size 1.27 1.27)
 				)
-				(hide yes)
+				(justify left)
 			)
 		)
-		(property "Value" "+5V"
-			(at 21.59 143.51 0)
+		(property "Value" "BC547"
+			(at 167.64 134.6199 0)
 			(effects
 				(font
 					(size 1.27 1.27)
 				)
+				(justify left)
 			)
 		)
-		(property "Footprint" ""
-			(at 21.59 138.43 0)
+		(property "Footprint" "Package_TO_SOT_THT:TO-92_Inline"
+			(at 167.64 135.255 0)
 			(effects
 				(font
 					(size 1.27 1.27)
+					(italic yes)
 				)
+				(justify left)
 				(hide yes)
 			)
 		)
-		(property "Datasheet" ""
-			(at 21.59 138.43 0)
+		(property "Datasheet" "https://www.onsemi.com/pub/Collateral/BC550-D.pdf"
+			(at 172.72 133.35 0)
 			(effects
 				(font
 					(size 1.27 1.27)
 				)
+				(justify left)
 				(hide yes)
 			)
 		)
-		(property "Description" "Power symbol creates a global label with name \"+5V\""
-			(at 21.59 138.43 0)
+		(property "Description" "0.1A Ic, 45V Vce, Small Signal NPN Transistor, TO-92"
+			(at 172.72 133.35 0)
 			(effects
 				(font
@@
 			)
 		)
+		(pin "3"
+		)
+		(pin "2"
+		)
 		(pin "1"
 		)
@@
 			(project "labRF"
 				(path "/2343659c-5e3e-4b93-ace6-06935e396af8"
-					(reference "#PWR07")
+					(reference "Q9")
 					(unit 1)
 				)
@@
 	)
 	(symbol
+		(lib_id "power:+3V3")
+		(at 21.59 138.43 180)
+		(unit 1)
+		(exclude_from_sim no)
+		(in_bom yes)
+		(on_board yes)
+		(dnp no)
+		(fields_autoplaced yes)
+		(property "Reference" "#PWR046"
+			(at 21.59 134.62 0)
+			(effects
+				(font
+					(size 1.27 1.27)
+				)
+				(hide yes)
+			)
+		)
+		(property "Value" "+3V3"
+			(at 21.59 143.51 0)
+			(effects
+				(font
+					(size 1.27 1.27)
+				)
+			)
+		)
+		(property "Footprint" ""
+			(at 21.59 138.43 0)
+			(effects
+				(font
+					(size 1.27 1.27)
+				)
+				(hide yes)
+			)
+		)
+		(property "Datasheet" ""
+			(at 21.59 138.43 0)
+			(effects
+				(font
+					(size 1.27 1.27)
+				)
+				(hide yes)
+			)
+		)
+		(property "Description" "Power symbol creates a global label with name \"+3V3\""
+			(at 21.59 138.43 0)
+			(effects
+				(font
+					(size 1.27 1.27)
+				)
+				(hide yes)
+			)
+		)
+		(pin "1"
+		)
+		(instances
+			(project "bluepill_design"
+				(path "/2343659c-5e3e-4b93-ace6-06935e396af8"
+					(reference "#PWR046")
+					(unit 1)
+				)
+			)
+		)
+	)
+	(symbol
 		(lib_id "power:GND")
 		(at 134.62 96.52 0)
@@
 				)
 			)
-		)
-	)
-	(symbol
-		(lib_id "power:+5V")
-		(at 21.59 161.29 180)
-		(unit 1)
-		(exclude_from_sim no)
-		(in_bom yes)
-		(on_board yes)
-		(dnp no)
-		(fields_autoplaced yes)
-		(property "Reference" "#PWR08"
-			(at 21.59 157.48 0)
-			(effects
-				(font
-					(size 1.27 1.27)
-				)
-				(hide yes)
-			)
-		)
-		(property "Value" "+5V"
-			(at 21.59 166.37 0)
-			(effects
-				(font
-					(size 1.27 1.27)
-				)
-			)
-		)
-		(property "Footprint" ""
-			(at 21.59 161.29 0)
-			(effects
-				(font
-					(size 1.27 1.27)
-				)
-				(hide yes)
-			)
-		)
-		(property "Datasheet" ""
-			(at 21.59 161.29 0)
-			(effects
-				(font
-					(size 1.27 1.27)
-				)
-				(hide yes)
-			)
-		)
-		(property "Description" "Power symbol creates a global label with name \"+5V\""
-			(at 21.59 161.29 0)
-			(effects
-				(font
-					(size 1.27 1.27)
-				)
-				(hide yes)
-			)
-		)
-		(pin "1"
-		)
-		(instances
-			(project "labRF"
-				(path "/2343659c-5e3e-4b93-ace6-06935e396af8"
-					(reference "#PWR08")
-					(unit 1)
-				)
-			)
